Commit message: Fixed URDF gantry_base_link origin

File: wsl_ws/src/aizee_model/urdf/aizee_urdf.urdf (robot description, URDF)
Before this commit: robot aizee_model, 24 links, 23 joints
Links:
- link base_link: mass None -> 8.72034111313672; geometry collision mesh filename=package://aizee_urdf/meshes/base_link.STL; visual mesh filename=package://aizee_urdf/meshes/base_link.STL
- link bl_wheel_link: geometry collision mesh filename=package://aizee_urdf/meshes/bl_wheel_link.STL; visual mesh filename=package://aizee_urdf/meshes/bl_wheel_link.STL
- link br_wheel_link: geometry collision mesh filename=package://aizee_urdf/meshes/br_wheel_link.STL; visual mesh filename=package://aizee_urdf/meshes/br_wheel_link.STL
- link fl_wheel_link: geometry collision mesh filename=package://aizee_urdf/meshes/fl_wheel_link.STL; visual mesh filename=package://aizee_urdf/meshes/fl_wheel_link.STL
- link fr_wheel_link: mass 0.426146379184825 -> 0.426146379184826; geometry collision mesh filename=package://aizee_urdf/meshes/fr_wheel_link.STL; visual mesh filename=package://aizee_urdf/meshes/fr_wheel_link.STL
- link gantry_base_link: mass 2.87751988356169 -> 2.87751988332943; geometry collision mesh filename=package://aizee_urdf/meshes/gantry_base_link.STL; visual mesh filename=package://aizee_urdf/meshes/gantry_base_link.STL
- link gantry_swivel_link: mass 4.14956251604638 -> 4.13256157024676; geometry collision mesh filename=package://aizee_urdf/meshes/gantry_swivel_link.STL; visual mesh filename=package://aizee_urdf/meshes/gantry_swivel_link.STL
- link head_pitch_link: mass 0.113884247586372 -> 0.113884247586373; geometry collision mesh filename=package://aizee_urdf/meshes/head_pitch_link.STL; visual mesh filename=package://aizee_urdf/meshes/head_pitch_link.STL
- link head_swivel_link: mass 0.0645692908984825 -> 0.0645692908984822; geometry collision mesh filename=package://aizee_urdf/meshes/head_swivel_link.STL; visual mesh filename=package://aizee_urdf/meshes/head_swivel_link.STL
- link head_tilt_link: geometry collision mesh filename=package://aizee_urdf/meshes/head_tilt_link.STL; visual mesh filename=package://aizee_urdf/meshes/head_tilt_link.STL
- link left_forearm_link: mass 0.133070486659464 -> 0.133070486658893; geometry collision mesh filename=package://aizee_urdf/meshes/left_forearm_link.STL; visual mesh filename=package://aizee_urdf/meshes/left_forearm_link.STL
- link left_lower_elbow_link: geometry collision mesh filename=package://aizee_urdf/meshes/left_lower_elbow_link.STL; visual mesh filename=package://aizee_urdf/meshes/left_lower_elbow_link.STL
- link left_shoulder_pitch_link: geometry collision mesh filename=package://aizee_urdf/meshes/left_shoulder_pitch_link.STL; visual mesh filename=package://aizee_urdf/meshes/left_shoulder_pitch_link.STL
- link left_upper_arm_link: geometry collision mesh filename=package://aizee_urdf/meshes/left_upper_arm_link.STL; visual mesh filename=package://aizee_urdf/meshes/left_upper_arm_link.STL
- link left_upper_elbow_link: mass 0.174638971892268 -> 0.174638971803144; geometry collision mesh filename=package://aizee_urdf/meshes/left_upper_elbow_link.STL; visual mesh filename=package://aizee_urdf/meshes/left_upper_elbow_link.STL
- link left_wrist_pitch_link: mass 0.0263062577407527 -> 0.0263062577407526; geometry collision mesh filename=package://aizee_urdf/meshes/left_wrist_pitch_link.STL; visual mesh filename=package://aizee_urdf/meshes/left_wrist_pitch_link.STL
- link left_wrist_tool_link: geometry collision mesh filename=package://aizee_urdf/meshes/left_wrist_tool_link.STL; visual mesh filename=package://aizee_urdf/meshes/left_wrist_tool_link.STL
- link right_forearm_link: mass 0.133069921434071 -> 0.133069921433842; geometry collision mesh filename=package://aizee_urdf/meshes/right_forearm_link.STL; visual mesh filename=package://aizee_urdf/meshes/right_forearm_link.STL
- link right_lower_elbow_link: geometry collision mesh filename=package://aizee_urdf/meshes/right_lower_elbow_link.STL; visual mesh filename=package://aizee_urdf/meshes/right_lower_elbow_link.STL
- link right_shoulder_pitch_link: geometry collision mesh filename=package://aizee_urdf/meshes/right_shoulder_pitch_link.STL; visual mesh filename=package://aizee_urdf/meshes/right_shoulder_pitch_link.STL
- link right_upper_arm_link: geometry collision mesh filename=package://aizee_urdf/meshes/right_upper_arm_link.STL; visual mesh filename=package://aizee_urdf/meshes/right_upper_arm_link.STL
- link right_upper_elbow_link: mass 0.17462194414463 -> 0.174621944055462; geometry collision mesh filename=package://aizee_urdf/meshes/right_upper_elbow_link.STL; visual mesh filename=package://aizee_urdf/meshes/right_upper_elbow_link.STL
- link right_wrist_pitch_link: geometry collision mesh filename=package://aizee_urdf/meshes/right_wrist_pitch_link.STL; visual mesh filename=package://aizee_urdf/meshes/right_wrist_pitch_link.STL
- link right_wrist_tool_link: geometry collision mesh filename=package://aizee_urdf/meshes/right_wrist_tool_link.STL; visual mesh filename=package://aizee_urdf/meshes/right_wrist_tool_link.STL
Joints:
- joint gantry_base_joint: origin xyz=-0.157321468199926 1.17368391308377 -0.309533448479469 rpy=0 0 0 -> xyz=0.0748880019266167 1.25057075528059 -0.106672907010273 rpy=0 0.940291533304643 0
- joint head_swivel_joint: origin xyz=0.242106081826129 0.135938295928873 2.97917338191868 rpy=2.20732432388274 0 -1.57079632679517 -> xyz=0.0134984733922502 0.0590514537320603 0.00240000000046037 rpy=-3.13556944999228 0 -1.57079632679489
- joint left_forearm_joint: limit lower=-2.0 upper=2.5 effort=1 velocity=1 -> lower=-3.14 upper=3.14 effort=1 velocity=1
- joint left_lower_elbow_joint: limit lower=-2.1 upper=0 effort=1 velocity=1 -> lower=-3.14 upper=3.14 effort=1 velocity=1
- joint left_shoulder_pitch_joint: limit lower=-1.82 upper=1.57 effort=1 velocity=1 -> lower=-3.14 upper=3.14 effort=1 velocity=1; origin xyz=0.0935898391350412 0.0585381329786352 2.88512198886941 rpy=-0.631198918193714 -0.0435891683503071 1.60263708973709 -> xyz=0.00190847339162745 -0.0183487092181731 -0.173009266509531 rpy=-1.5707963267949 0 1.6247704646502
- joint left_upper_arm_joint: limit lower=-2.7 upper=0 effort=1 velocity=1 -> lower=-3.14 upper=3.14 effort=1 velocity=1
- joint left_upper_elbow_joint: limit lower=-0.815 upper=1.05 effort=1 velocity=1 -> lower=-3.14 upper=3.14 effort=1 velocity=1
- joint left_wrist_pitch_joint: limit lower=-0.22 upper=0.22 effort=1 velocity=1 -> lower=-3.14 upper=3.14 effort=1 velocity=1
- joint left_wrist_tool_joint: limit lower=-1.5 upper=1.5 effort=1 velocity=1 -> lower=-3.14 upper=3.14 effort=1 velocity=1
- joint right_forearm_joint: limit lower=-2.5 upper=2.0 effort=1 velocity=1 -> lower=-3.14 upper=3.14 effort=1 velocity=1
- joint right_lower_elbow_joint: limit lower=0 upper=2.1 effort=1 velocity=1 -> lower=-3.14 upper=3.14 effort=1 velocity=1
- joint right_shoulder_pitch_joint: limit lower=1.57 upper=1.82 effort=1 velocity=1 -> lower=-3.14 upper=3.14 effort=1 velocity=1; origin xyz=0.274293991616603 0.058538132978631 3.01701581020399 rpy=2.51039373539614 -0.0435891683503091 1.60263708973709 -> xyz=0.00190847339150882 -0.0183487092181824 0.0507092415096265 rpy=1.57079632679496 0 1.6247704646502
- joint right_upper_arm_joint: limit lower=0 upper=2.7 effort=1 velocity=1 -> lower=-3.14 upper=3.14 effort=1 velocity=1
- joint right_upper_elbow_joint: limit lower=-1.05 upper=0.815 effort=1 velocity=1 -> lower=-3.14 upper=3.14 effort=1 velocity=1
- joint right_wrist_pitch_joint: limit lower=-0.22 upper=0.22 effort=1 velocity=1 -> lower=-3.14 upper=3.14 effort=1 velocity=1
- joint right_wrist_tool_joint: limit lower=-1.5 upper=1.5 effort=1 velocity=1 -> lower=-3.14 upper=3.14 effort=1 velocity=1

Commit message: Removed inertial data from base_link

File: wsl_ws/src/aizee_model/urdf/aizee_urdf.urdf (robot description, URDF)
Before this commit: robot aizee_urdf, 24 links, 23 joints
Links:
- link base_link: mass 8.72034111313672 -> None
