Commit message: Moveit servo working, TF links are off, preventing good kinematics for servo.

File: wsl_ws/src/aizee_model/urdf/aizee_model.urdf (robot description, URDF)
Before this commit: robot aizee_model, 24 links, 23 joints
Links:
- link base_link: mass 8.83294978683653 -> None
Joints:
- joint gantry_base_joint: origin xyz=-0.157321468199926 1.17368391308377 -3.09533448479469 rpy=0 0 0 -> xyz=-0.157321468199926 1.17368391308377 -0.309533448479469 rpy=0 0 0
- joint left_shoulder_pitch_joint: axis 0 1 0 -> 0 -1 0
- joint left_upper_arm_joint: axis 0.0539479353612052 0 0.998543749802813 -> -0.0539479353612052 0 -0.998543749802813
- joint left_upper_elbow_joint: axis 0 1 0 -> 0 -1 0
- joint left_wrist_pitch_joint: axis 0 0.866025403784494 -0.499999999999905 -> 0 -0.866025403784494 0.499999999999905
- joint right_shoulder_pitch_joint: axis 0 1 0 -> 0 -1 0
- joint right_upper_arm_joint: axis 0.0539479353612056 0 -0.998543749802813 -> -0.0539479353612056 0 0.998543749802813
- joint right_upper_elbow_joint: axis 0 1 0 -> 0 -1 0
- joint right_wrist_pitch_joint: axis 0 0.999999999998175 0 -> 0 -0.999999999998175 0
- joint right_wrist_tool_joint: axis 0.995843763645616 0.09048526345698 -0.0103737893393006 -> -0.995843763645616 -0.09048526345698 0.0103737893393006

File: wsl_ws/src/moveit_aizee/config/aizee_model.ros2_control.xacro (robot description, xacro)
@@ -1,17 +1,26 @@
 <?xml version="1.0"?>
 <robot xmlns:xacro="http://www.ros.org/wiki/xacro">
-  <xacro:macro name="aizee_model_ros2_control" params="name initial_positions_file">
-    <xacro:property name="initial_positions" value="${load_yaml(initial_positions_file)['initial_positions']}"/>
+  <!-- === aizee_model_ros2_control ======================================== -->
+  <xacro:macro name="aizee_model_ros2_control"
+               params="name hardware_type initial_positions_file">
+    <!-- initial positions for simulation -->
+    <xacro:property name="initial_positions"
+                    value="${load_yaml(initial_positions_file)['initial_positions']}" />
     <ros2_control name="${name}" type="system">
       <hardware>
+        <xacro:if value="${hardware_type == 'mock_components'}">
+          <plugin>ros2_control_demo_hardware/MockSystem</plugin>
+        </xacro:if>
+        <xacro:unless value="${hardware_type == 'mock_components'}">
           <plugin>feetech_ros2_driver/FeetechHardwareInterface</plugin>
-          <param name="usb_port">/dev/ttyUSB0</param> <!-- required -->
-          <param name="baudrate">1000000</param>     <!-- optional -->
+          <param name="usb_port">/dev/ttyUSB0</param>
+          <param name="baudrate">1000000</param>
+        </xacro:unless>
       </hardware>
-      <!-- Joint definitions -->
-      <xacro:macro name="feetech_joint" params="joint_name id">
+      <!-- helper macro: *offset* defaults to 0 -->
+      <xacro:macro name="feetech_joint" params="joint_name id offset:=0">
         <joint name="${joint_name}">
           <param name="id">${id}</param>
-          <param name="offset">0</param>
+          <param name="offset">${offset}</param>
           <param name="p_cofficient">16</param>
           <param name="d_cofficient">8</param>
@@ -23,20 +32,20 @@
         </joint>
       </xacro:macro>
-      <!-- Left Arm Joints -->
-      <xacro:feetech_joint joint_name="left_shoulder_pitch_joint" id="11"/>
-      <xacro:feetech_joint joint_name="left_upper_arm_joint" id="12"/>
-      <xacro:feetech_joint joint_name="left_upper_elbow_joint" id="13"/>
-      <xacro:feetech_joint joint_name="left_lower_elbow_joint" id="14"/>
-      <xacro:feetech_joint joint_name="left_forearm_joint" id="15"/>
-      <xacro:feetech_joint joint_name="left_wrist_pitch_joint" id="16"/>
-      <xacro:feetech_joint joint_name="left_wrist_tool_joint" id="17"/>
-      <!-- Right Arm Joints -->
-      <xacro:feetech_joint joint_name="right_shoulder_pitch_joint" id="1"/>
-      <xacro:feetech_joint joint_name="right_upper_arm_joint" id="2"/>
-      <xacro:feetech_joint joint_name="right_upper_elbow_joint" id="3"/>
-      <xacro:feetech_joint joint_name="right_lower_elbow_joint" id="4"/>
-      <xacro:feetech_joint joint_name="right_forearm_joint" id="5"/>
-      <xacro:feetech_joint joint_name="right_wrist_pitch_joint" id="6"/>
-      <xacro:feetech_joint joint_name="right_wrist_tool_joint" id="7"/>
+      <!-- ── Left Arm (measured offsets) ─────────────────────────────────── -->
+      <xacro:feetech_joint joint_name="left_shoulder_pitch_joint" id="11" offset="1800" />
+      <xacro:feetech_joint joint_name="left_upper_arm_joint"      id="12" offset="1200" />
+      <xacro:feetech_joint joint_name="left_upper_elbow_joint"    id="13" offset="1400" />
+      <xacro:feetech_joint joint_name="left_lower_elbow_joint"    id="14" offset="-2100" />
+      <xacro:feetech_joint joint_name="left_forearm_joint"        id="15" offset="-2400" />
+      <xacro:feetech_joint joint_name="left_wrist_pitch_joint"    id="16" offset="-1700" />
+      <xacro:feetech_joint joint_name="left_wrist_tool_joint"     id="17" offset="1800" />
+      <!-- ── Right Arm (measured offsets) ────────────────────────────────── -->
+      <xacro:feetech_joint joint_name="right_shoulder_pitch_joint" id="1" offset="-1600"/>
+      <xacro:feetech_joint joint_name="right_upper_arm_joint"      id="2" offset="2300" />
+      <xacro:feetech_joint joint_name="right_upper_elbow_joint"    id="3" offset="-1000" />
+      <xacro:feetech_joint joint_name="right_lower_elbow_joint"    id="4" offset="2500" />
+      <xacro:feetech_joint joint_name="right_forearm_joint"        id="5" offset="-1400" />
+      <xacro:feetech_joint joint_name="right_wrist_pitch_joint"    id="6" offset="1250" />
+      <xacro:feetech_joint joint_name="right_wrist_tool_joint"     id="7" offset="-1800" />
     </ros2_control>
   </xacro:macro>

File: wsl_ws/src/moveit_aizee/config/aizee_model.urdf.xacro (robot description, xacro)
@@ -1,5 +1,5 @@
 <?xml version="1.0"?>
 <robot xmlns:xacro="http://www.ros.org/wiki/xacro" name="aizee_model">
-    <xacro:arg name="ros2_control_hardware_type" default="mock_components"/>
+    <xacro:arg name="ros2_control_hardware_type" default="feetech"/>
     <xacro:arg name="initial_positions_file" default="initial_positions.yaml" />
     <!-- Import aizee_model urdf file -->
@@ -7,4 +7,7 @@
     <!-- Import control_xacro -->
     <xacro:include filename="aizee_model.ros2_control.xacro" />
-    <xacro:aizee_model_ros2_control name="$(arg ros2_control_hardware_type)" initial_positions_file="$(arg initial_positions_file)"/>
+    <xacro:aizee_model_ros2_control
+          name="aizee_hw"
+          hardware_type="$(arg ros2_control_hardware_type)"
+          initial_positions_file="$(arg initial_positions_file)"/>
 </robot>

Commit message: Fixed URDF names.

File: wsl_ws/src/aizee_model/urdf/aizee_model.urdf (robot description, URDF)
Before this commit: robot aizee_urdf, 24 links, 23 joints
Links:
- link base_link: geometry collision mesh filename=package://aizee_model/meshes/base_link.STL; visual mesh filename=package://aizee_model/meshes/base_link.STL
- link bl_wheel_link: geometry collision mesh filename=package://aizee_model/meshes/bl_wheel_link.STL; visual mesh filename=package://aizee_model/meshes/bl_wheel_link.STL
- link br_wheel_link: geometry collision mesh filename=package://aizee_model/meshes/br_wheel_link.STL; visual mesh filename=package://aizee_model/meshes/br_wheel_link.STL
- link fl_wheel_link: geometry collision mesh filename=package://aizee_model/meshes/fl_wheel_link.STL; visual mesh filename=package://aizee_model/meshes/fl_wheel_link.STL
- link fr_wheel_link: geometry collision mesh filename=package://aizee_model/meshes/fr_wheel_link.STL; visual mesh filename=package://aizee_model/meshes/fr_wheel_link.STL
- link gantry_base_link: geometry collision mesh filename=package://aizee_model/meshes/gantry_base_link.STL; visual mesh filename=package://aizee_model/meshes/gantry_base_link.STL
- link gantry_swivel_link: geometry collision mesh filename=package://aizee_model/meshes/gantry_swivel_link.STL; visual mesh filename=package://aizee_model/meshes/gantry_swivel_link.STL
- link head_pitch_link: geometry collision mesh filename=package://aizee_model/meshes/head_pitch_link.STL; visual mesh filename=package://aizee_model/meshes/head_pitch_link.STL
- link head_swivel_link: geometry collision mesh filename=package://aizee_model/meshes/head_swivel_link.STL; visual mesh filename=package://aizee_model/meshes/head_swivel_link.STL
- link head_tilt_link: geometry collision mesh filename=package://aizee_model/meshes/head_tilt_link.STL; visual mesh filename=package://aizee_model/meshes/head_tilt_link.STL
- link left_forearm_link: geometry collision mesh filename=package://aizee_model/meshes/left_forearm_link.STL; visual mesh filename=package://aizee_model/meshes/left_forearm_link.STL
- link left_lower_elbow_link: geometry collision mesh filename=package://aizee_model/meshes/left_lower_elbow_link.STL; visual mesh filename=package://aizee_model/meshes/left_lower_elbow_link.STL
- link left_shoulder_pitch_link: geometry collision mesh filename=package://aizee_model/meshes/left_shoulder_pitch_link.STL; visual mesh filename=package://aizee_model/meshes/left_shoulder_pitch_link.STL
- link left_upper_arm_link: geometry collision mesh filename=package://aizee_model/meshes/left_upper_arm_link.STL; visual mesh filename=package://aizee_model/meshes/left_upper_arm_link.STL
- link left_upper_elbow_link: geometry collision mesh filename=package://aizee_model/meshes/left_upper_elbow_link.STL; visual mesh filename=package://aizee_model/meshes/left_upper_elbow_link.STL
- link left_wrist_pitch_link: geometry collision mesh filename=package://aizee_model/meshes/left_wrist_pitch_link.STL; visual mesh filename=package://aizee_model/meshes/left_wrist_pitch_link.STL
- link left_wrist_tool_link: geometry collision mesh filename=package://aizee_model/meshes/left_wrist_tool_link.STL; visual mesh filename=package://aizee_model/meshes/left_wrist_tool_link.STL
- link right_forearm_link: geometry collision mesh filename=package://aizee_model/meshes/right_forearm_link.STL; visual mesh filename=package://aizee_model/meshes/right_forearm_link.STL
- link right_lower_elbow_link: geometry collision mesh filename=package://aizee_model/meshes/right_lower_elbow_link.STL; visual mesh filename=package://aizee_model/meshes/right_lower_elbow_link.STL
- link right_shoulder_pitch_link: geometry collision mesh filename=package://aizee_model/meshes/right_shoulder_pitch_link.STL; visual mesh filename=package://aizee_model/meshes/right_shoulder_pitch_link.STL
- link right_upper_arm_link: geometry collision mesh filename=package://aizee_model/meshes/right_upper_arm_link.STL; visual mesh filename=package://aizee_model/meshes/right_upper_arm_link.STL
- link right_upper_elbow_link: geometry collision mesh filename=package://aizee_model/meshes/right_upper_elbow_link.STL; visual mesh filename=package://aizee_model/meshes/right_upper_elbow_link.STL
- link right_wrist_pitch_link: geometry collision mesh filename=package://aizee_model/meshes/right_wrist_pitch_link.STL; visual mesh filename=package://aizee_model/meshes/right_wrist_pitch_link.STL
- link right_wrist_tool_link: geometry collision mesh filename=package://aizee_model/meshes/right_wrist_tool_link.STL; visual mesh filename=package://aizee_model/meshes/right_wrist_tool_link.STL

Commit message: Fixed origins... again.

File: wsl_ws/src/aizee_model/urdf/aizee_model.urdf (robot description, URDF)
Before this commit: robot aizee_model, 24 links, 23 joints
Links:
- link base_link: mass None -> 8.72034111313673
- link fl_wheel_link: mass 0.426146379160631 -> 0.426146379160632
- link fr_wheel_link: mass 0.426146379184826 -> 0.426146379184825
- link gantry_base_link: mass 2.87751988332943 -> 2.87751988360274
- link gantry_swivel_link: mass 4.13256157024676 -> 4.13256156537212
- link head_pitch_link: mass 0.113884247586373 -> 0.113884246009613
- link head_swivel_link: mass 0.0645692908984822 -> 0.0645692908984826
- link left_forearm_link: mass 0.133070486658893 -> 0.133070486458284
- link left_lower_elbow_link: mass 0.151902535776002 -> 0.151902535663641
- link left_shoulder_pitch_link: mass 0.224603058456901 -> 0.224603056164951
- link left_upper_arm_link: mass 0.311240729701745 -> 0.311240459874834
- link left_upper_elbow_link: mass 0.174638971803144 -> 0.174639013065772
- link left_wrist_pitch_link: mass 0.0263062577407526 -> 0.0263062310477304
- link right_forearm_link: mass 0.133069921433842 -> 0.133069689452656
- link right_lower_elbow_link: mass 0.151904197101514 -> 0.151904197101513
- link right_shoulder_pitch_link: mass 0.2246031087904 -> 0.224603105390766
- link right_upper_arm_link: mass 0.311238424356508 -> 0.311239451264541
- link right_upper_elbow_link: mass 0.174621944055462 -> 0.17462194427021
- link right_wrist_pitch_link: mass 0.0263065978280762 -> 0.0263065913042516
Joints:
- joint gantry_base_joint: origin xyz=0.0748880019266167 1.25057075528059 -0.106672907010273 rpy=0 0.940291533304643 0 -> xyz=8.0773E-05 1.1737 5.8955E-05 rpy=3.1416 -0.94029 -3.1416
- joint gantry_swivel_joint: origin xyz=-0.00171500001182112 0 0.0449999999986612 rpy=1.57079632679467 0 2.20130112028515 -> xyz=-0.001715 0 0.045 rpy=1.5708 0 2.2013
- joint head_pitch_joint: origin xyz=-0.00715658863949598 0 0.000220485265825118 rpy=0.0301375093124696 -0.0107085179536229 1.06890143125903 -> xyz=-0.00715658863950375 0 0.000220485265838899 rpy=0.0301375093124696 -0.0107085179536229 1.06890143125903
- joint head_swivel_joint: origin xyz=0.0134984733922502 0.0590514537320603 0.00240000000046037 rpy=-3.13556944999228 0 -1.57079632679489 -> xyz=-0.14381 0.13594 0.0001 rpy=0.0060232 0 -1.5708
- joint head_tilt_joint: origin xyz=-0.0428400156095763 0 0 rpy=0 -0.0307989676412341 0.000185569376448724 -> xyz=-0.0428400156095683 0 0 rpy=0 -0.0307989676412341 0.000185569376448724
- joint left_forearm_joint: axis 0.980643317783864 -0.0724305556359989 0.181913435172108 -> 0.980643317783876 -0.0724305556359773 0.18191343517205; origin xyz=-0.0269534702231413 -0.00214213478108545 -0.00613953045680382 rpy=-2.03700008275405 -0.274733744913231 -0.191545917444499 -> xyz=-0.0269534702231389 -0.00214213478108321 -0.00613953045680213 rpy=-2.03700008275405 -0.274733744913246 -0.191545917444494
- joint left_lower_elbow_joint: axis 0.0880130878902615 0.920101163566549 -0.381664178517586 -> 0.0880130878903102 0.920101163566567 -0.381664178517532; origin xyz=0.0381999999999998 0.112403218450234 0 rpy=1.96400162440634 -0.0881271151701579 -1.59563952845257 -> xyz=0.0381999999999999 0.112403218450237 0 rpy=1.96400162440628 -0.0881271151702069 -1.59563952845257
- joint left_shoulder_pitch_joint: axis 0 -1 0 -> 0 1 0; origin xyz=0.00190847339162745 -0.0183487092181731 -0.173009266509531 rpy=-1.5707963267949 0 1.6247704646502 -> xyz=-0.132221795513797 0.0585381329785393 0.0484092415095189 rpy=1.57079632679485 0 1.51682218893965
- joint left_upper_arm_joint: axis -0.0539479353612052 0 -0.998543749802813 -> 0.0539479353612109 0 0.998543749802813; origin xyz=0 -0.0210000249999997 0 rpy=0.0081422452723712 -0.00061707146343348 0.151282779582159 -> xyz=0 0.106100000000015 0 rpy=0.00814224527237571 -0.000617071463435104 0.151282779582204
- joint left_upper_elbow_joint: axis 0 -1 0 -> 0 1 0; origin xyz=-0.0862752361730879 0.0131904590673325 0.00456101284018645 rpy=1.72230140662095 1.51682218893959 3.1415926535897 -> xyz=-0.0862752361730876 0.0131904590673321 0.00456101284012125 rpy=1.72230140661996 1.51682218893961 3.14159265358868
- joint left_wrist_pitch_joint: axis 0 -0.866025403784494 0.499999999999905 -> 0 0.866025403784494 -0.499999999999905; origin xyz=-0.124566694244266 0.00920052654643683 -0.0231076425516821 rpy=3.08769993659024 -1.35192984023634 -2.62673064646431 -> xyz=-0.124566694244269 0.00920052654643505 -0.0231076425516841 rpy=3.08769993658993 -1.35192984023637 -2.62673064646398
- joint left_wrist_tool_joint: axis 0.995843763645561 0.0904852634575847 -0.0103737893393016 -> 0.995843763645555 0.0904852634576426 -0.0103737893393476; origin xyz=0 0.0141339745962043 0.0264807621135394 rpy=-2.07922112326353 -0.0741625565420776 0.0531350305034689 -> xyz=0 0.0141339745962058 0.0264807621135386 rpy=-2.07922112326353 -0.0741625565421061 0.0531350305035374
- joint right_forearm_joint: axis 0.980643317783807 -0.0724305556360285 -0.181913435172403 -> 0.980643317783738 -0.0724305556360726 -0.181913435172757; origin xyz=-0.0269534702231529 -0.00214213478108295 0.00613953045680563 rpy=2.03700008275405 0.274733744913234 -0.1915459174445 -> xyz=-0.0269534702231089 -0.00214213478098909 0.00613953045678181 rpy=2.03700008275405 0.274733744913229 -0.191545917444501
- joint right_lower_elbow_joint: axis 0.0880130878899545 0.920101163566575 0.381664178517595 -> 0.0880130878895927 0.920101163566584 0.381664178517656; origin xyz=0.0381999999999999 0.112403218450209 0 rpy=-1.96400162440628 0.0881271151698512 -1.59563952845255 -> xyz=0.0382000000000001 0.112403218450237 0 rpy=-1.96400162440639 0.0881271151694865 -1.59563952845256
- joint right_shoulder_pitch_joint: axis 0 -1 0 -> 0 1 0; origin xyz=0.00190847339150882 -0.0183487092181824 0.0507092415096265 rpy=1.57079632679496 0 1.6247704646502 -> xyz=-0.132221795513731 0.0585381329786272 -0.0482092415089532 rpy=-1.57079632679482 0 1.51682218893965
- joint right_upper_arm_joint: axis -0.0539479353612056 0 0.998543749802813 -> 0.0539479353612105 0 -0.998543749802813; origin xyz=0 0.106100000000005 0 rpy=-0.00814224527238941 0.000617071463436487 0.151282779581843 -> xyz=0 0.106100000000039 0 rpy=-0.00814224527237025 0.000617071463434093 0.151282779581485
- joint right_upper_elbow_joint: axis 0 -1 0 -> 0 1 0; origin xyz=-0.0837801498896911 0.0128131437121982 -0.00493341280181048 rpy=-1.7223014066196 -1.5168221889396 3.14159265358868 -> xyz=-0.0837801498896704 0.012813143712194 -0.00493341280167864 rpy=-1.72230140661924 -1.5168221889396 3.14159265358867
- joint right_wrist_pitch_joint: axis 0 -0.999999999998175 0 -> 0 1 0; origin xyz=-0.124566694244255 0.00920052654643555 0.0231076425516814 rpy=2.56409921497058 -1.35192985229203 0.514862043305627 -> xyz=-0.124566694244279 0.00920052654645065 0.0231076425517911 rpy=-0.577491492596529 -1.35192984023572 0.514862007124234
- joint right_wrist_tool_joint: axis -0.995843763645616 -0.09048526345698 0.0103737893393006 -> 0.99584376364562 0.0904852634569211 -0.0103737893393444; origin xyz=0 0.00100005732113667 -0.0299999980892369 rpy=1.58753777306352 0.0907744300301574 3.13273498556734 -> xyz=0 -0.000999999999963808 0.03 rpy=-1.5540529618699 -0.0907744325651698 -3.13273515949314

Commit message: Fixed directions and origins... again...

File: wsl_ws/src/aizee_model/urdf/aizee_model.urdf (robot description, URDF)
Before this commit: robot aizee_model, 24 links, 23 joints
Links:
- link base_link: mass 8.72034111313673 -> None
Joints:
- joint left_shoulder_pitch_joint: axis 0 1 0 -> 0 -1 0
- joint left_upper_arm_joint: axis 0.0539479353612109 0 0.998543749802813 -> -0.0539479353612109 0 -0.998543749802813
- joint left_upper_elbow_joint: axis 0 1 0 -> 0 -1 0
- joint left_wrist_pitch_joint: axis 0 0.866025403784494 -0.499999999999905 -> 0 -0.866025403784494 0.499999999999905
- joint right_shoulder_pitch_joint: axis 0 1 0 -> 0 -1 0
- joint right_upper_arm_joint: axis 0.0539479353612105 0 -0.998543749802813 -> -0.0539479353612105 0 0.998543749802813
- joint right_upper_elbow_joint: axis 0 1 0 -> 0 -1 0
- joint right_wrist_pitch_joint: axis 0 1 0 -> 0 -1 0
- joint right_wrist_tool_joint: axis 0.99584376364562 0.0904852634569211 -0.0103737893393444 -> -0.99584376364562 -0.0904852634569211 0.0103737893393444
