Commit message: Setup Moveit servo: use-> ros2 launch moveit_aizee servo.launch.py

File: wsl_ws/install/moveit_aizee/share/moveit_aizee/config/aizee_model.ros2_control.xacro (robot description, xacro)
@@ -1,110 +1 @@
-<?xml version="1.0"?>
-<robot xmlns:xacro="http://www.ros.org/wiki/xacro">
-    <xacro:macro name="aizee_model_ros2_control" params="name initial_positions_file">
-        <xacro:property name="initial_positions" value="${load_yaml(initial_positions_file)['initial_positions']}"/>
-        <ros2_control name="${name}" type="system">
-            <hardware>
-                <!-- By default, set up controllers for simulation. This won't work on real hardware -->
-                <plugin>mock_components/GenericSystem</plugin>
-            </hardware>
-            <joint name="left_shoulder_pitch_joint">
-                <command_interface name="position"/>
-                <state_interface name="position">
-                  <param name="initial_value">${initial_positions['left_shoulder_pitch_joint']}</param>
-                </state_interface>
-                <state_interface name="velocity"/>
-            </joint>
-            <joint name="left_upper_arm_joint">
-                <command_interface name="position"/>
-                <state_interface name="position">
-                  <param name="initial_value">${initial_positions['left_upper_arm_joint']}</param>
-                </state_interface>
-                <state_interface name="velocity"/>
-            </joint>
-            <joint name="left_upper_elbow_joint">
-                <command_interface name="position"/>
-                <state_interface name="position">
-                  <param name="initial_value">${initial_positions['left_upper_elbow_joint']}</param>
-                </state_interface>
-                <state_interface name="velocity"/>
-            </joint>
-            <joint name="left_lower_elbow_joint">
-                <command_interface name="position"/>
-                <state_interface name="position">
-                  <param name="initial_value">${initial_positions['left_lower_elbow_joint']}</param>
-                </state_interface>
-                <state_interface name="velocity"/>
-            </joint>
-            <joint name="left_forearm_joint">
-                <command_interface name="position"/>
-                <state_interface name="position">
-                  <param name="initial_value">${initial_positions['left_forearm_joint']}</param>
-                </state_interface>
-                <state_interface name="velocity"/>
-            </joint>
-            <joint name="left_wrist_pitch_joint">
-                <command_interface name="position"/>
-                <state_interface name="position">
-                  <param name="initial_value">${initial_positions['left_wrist_pitch_joint']}</param>
-                </state_interface>
-                <state_interface name="velocity"/>
-            </joint>
-            <joint name="left_wrist_tool_joint">
-                <command_interface name="position"/>
-                <state_interface name="position">
-                  <param name="initial_value">${initial_positions['left_wrist_tool_joint']}</param>
-                </state_interface>
-                <state_interface name="velocity"/>
-            </joint>
-            <joint name="right_shoulder_pitch_joint">
-                <command_interface name="position"/>
-                <state_interface name="position">
-                  <param name="initial_value">${initial_positions['right_shoulder_pitch_joint']}</param>
-                </state_interface>
-                <state_interface name="velocity"/>
-            </joint>
-            <joint name="right_upper_arm_joint">
-                <command_interface name="position"/>
-                <state_interface name="position">
-                  <param name="initial_value">${initial_positions['right_upper_arm_joint']}</param>
-                </state_interface>
-                <state_interface name="velocity"/>
-            </joint>
-            <joint name="right_upper_elbow_joint">
-                <command_interface name="position"/>
-                <state_interface name="position">
-                  <param name="initial_value">${initial_positions['right_upper_elbow_joint']}</param>
-                </state_interface>
-                <state_interface name="velocity"/>
-            </joint>
-            <joint name="right_lower_elbow_joint">
-                <command_interface name="position"/>
-                <state_interface name="position">
-                  <param name="initial_value">${initial_positions['right_lower_elbow_joint']}</param>
-                </state_interface>
-                <state_interface name="velocity"/>
-            </joint>
-            <joint name="right_forearm_joint">
-                <command_interface name="position"/>
-                <state_interface name="position">
-                  <param name="initial_value">${initial_positions['right_forearm_joint']}</param>
-                </state_interface>
-                <state_interface name="velocity"/>
-            </joint>
-            <joint name="right_wrist_pitch_joint">
-                <command_interface name="position"/>
-                <state_interface name="position">
-                  <param name="initial_value">${initial_positions['right_wrist_pitch_joint']}</param>
-                </state_interface>
-                <state_interface name="velocity"/>
-            </joint>
-            <joint name="right_wrist_tool_joint">
-                <command_interface name="position"/>
-                <state_interface name="position">
-                  <param name="initial_value">${initial_positions['right_wrist_tool_joint']}</param>
-                </state_interface>
-                <state_interface name="velocity"/>
-            </joint>
-        </ros2_control>
-    </xacro:macro>
-</robot>
+/home/ltr/aizee/wsl_ws/src/moveit_aizee/config/aizee_model.ros2_control.xacro

File: wsl_ws/install/moveit_aizee/share/moveit_aizee/config/aizee_model.urdf.xacro (robot description, xacro)
@@ -1,9 +1 @@
-<?xml version="1.0"?>
-<robot xmlns:xacro="http://www.ros.org/wiki/xacro" name="aizee_model">
-    <xacro:arg name="initial_positions_file" default="initial_positions.yaml" />
-    <!-- Import aizee_model urdf file -->
-    <xacro:include filename="$(find aizee_model)/urdf/aizee_model.urdf" />
-    <!-- Import control_xacro -->
-    <xacro:include filename="aizee_model.ros2_control.xacro" />
-    <xacro:aizee_model_ros2_control name="FakeSystem" initial_positions_file="$(arg initial_positions_file)"/>
-</robot>
+/home/ltr/aizee/wsl_ws/src/moveit_aizee/config/aizee_model.urdf.xacro

File: wsl_ws/src/moveit_aizee/config/aizee_model.ros2_control.xacro (robot description, xacro)
@@ -1,110 +1,43 @@
 <?xml version="1.0"?>
 <robot xmlns:xacro="http://www.ros.org/wiki/xacro">
-    <xacro:macro name="aizee_model_ros2_control" params="name initial_positions_file">
-        <xacro:property name="initial_positions" value="${load_yaml(initial_positions_file)['initial_positions']}"/>
-        <ros2_control name="${name}" type="system">
-            <hardware>
-                <!-- By default, set up controllers for simulation. This won't work on real hardware -->
-                <plugin>mock_components/GenericSystem</plugin>
-            </hardware>
-            <joint name="left_shoulder_pitch_joint">
-                <command_interface name="position"/>
-                <state_interface name="position">
-                  <param name="initial_value">${initial_positions['left_shoulder_pitch_joint']}</param>
-                </state_interface>
-                <state_interface name="velocity"/>
-            </joint>
-            <joint name="left_upper_arm_joint">
-                <command_interface name="position"/>
-                <state_interface name="position">
-                  <param name="initial_value">${initial_positions['left_upper_arm_joint']}</param>
-                </state_interface>
-                <state_interface name="velocity"/>
-            </joint>
-            <joint name="left_upper_elbow_joint">
-                <command_interface name="position"/>
-                <state_interface name="position">
-                  <param name="initial_value">${initial_positions['left_upper_elbow_joint']}</param>
-                </state_interface>
-                <state_interface name="velocity"/>
-            </joint>
-            <joint name="left_lower_elbow_joint">
-                <command_interface name="position"/>
-                <state_interface name="position">
-                  <param name="initial_value">${initial_positions['left_lower_elbow_joint']}</param>
-                </state_interface>
-                <state_interface name="velocity"/>
-            </joint>
-            <joint name="left_forearm_joint">
-                <command_interface name="position"/>
-                <state_interface name="position">
-                  <param name="initial_value">${initial_positions['left_forearm_joint']}</param>
-                </state_interface>
-                <state_interface name="velocity"/>
-            </joint>
-            <joint name="left_wrist_pitch_joint">
-                <command_interface name="position"/>
-                <state_interface name="position">
-                  <param name="initial_value">${initial_positions['left_wrist_pitch_joint']}</param>
-                </state_interface>
-                <state_interface name="velocity"/>
-            </joint>
-            <joint name="left_wrist_tool_joint">
-                <command_interface name="position"/>
-                <state_interface name="position">
-                  <param name="initial_value">${initial_positions['left_wrist_tool_joint']}</param>
-                </state_interface>
-                <state_interface name="velocity"/>
-            </joint>
-            <joint name="right_shoulder_pitch_joint">
-                <command_interface name="position"/>
-                <state_interface name="position">
-                  <param name="initial_value">${initial_positions['right_shoulder_pitch_joint']}</param>
-                </state_interface>
-                <state_interface name="velocity"/>
-            </joint>
-            <joint name="right_upper_arm_joint">
-                <command_interface name="position"/>
-                <state_interface name="position">
-                  <param name="initial_value">${initial_positions['right_upper_arm_joint']}</param>
-                </state_interface>
-                <state_interface name="velocity"/>
-            </joint>
-            <joint name="right_upper_elbow_joint">
-                <command_interface name="position"/>
-                <state_interface name="position">
-                  <param name="initial_value">${initial_positions['right_upper_elbow_joint']}</param>
-                </state_interface>
-                <state_interface name="velocity"/>
-            </joint>
-            <joint name="right_lower_elbow_joint">
-                <command_interface name="position"/>
-                <state_interface name="position">
-                  <param name="initial_value">${initial_positions['right_lower_elbow_joint']}</param>
-                </state_interface>
-                <state_interface name="velocity"/>
-            </joint>
-            <joint name="right_forearm_joint">
-                <command_interface name="position"/>
-                <state_interface name="position">
-                  <param name="initial_value">${initial_positions['right_forearm_joint']}</param>
-                </state_interface>
-                <state_interface name="velocity"/>
-            </joint>
-            <joint name="right_wrist_pitch_joint">
-                <command_interface name="position"/>
-                <state_interface name="position">
-                  <param name="initial_value">${initial_positions['right_wrist_pitch_joint']}</param>
-                </state_interface>
-                <state_interface name="velocity"/>
-            </joint>
-            <joint name="right_wrist_tool_joint">
-                <command_interface name="position"/>
-                <state_interface name="position">
-                  <param name="initial_value">${initial_positions['right_wrist_tool_joint']}</param>
-                </state_interface>
-                <state_interface name="velocity"/>
-            </joint>
-        </ros2_control>
-    </xacro:macro>
+  <xacro:macro name="aizee_model_ros2_control" params="name initial_positions_file">
+    <xacro:property name="initial_positions" value="${load_yaml(initial_positions_file)['initial_positions']}"/>
+    <ros2_control name="${name}" type="system">
+      <hardware>
+          <plugin>feetech_ros2_driver/FeetechHardwareInterface</plugin>
+          <param name="usb_port">/dev/ttyUSB0</param> <!-- required -->
+          <param name="baudrate">1000000</param>     <!-- optional -->
+      </hardware>
+      <!-- Joint definitions -->
+      <xacro:macro name="feetech_joint" params="joint_name id">
+        <joint name="${joint_name}">
+          <param name="id">${id}</param>
+          <param name="offset">0</param>
+          <param name="p_cofficient">16</param>
+          <param name="d_cofficient">8</param>
+          <command_interface name="position"/>
+          <state_interface name="position">
+            <param name="initial_value">${initial_positions[joint_name]}</param>
+          </state_interface>
+          <state_interface name="velocity"/>
+        </joint>
+      </xacro:macro>
+      <!-- Left Arm Joints -->
+      <xacro:feetech_joint joint_name="left_shoulder_pitch_joint" id="11"/>
+      <xacro:feetech_joint joint_name="left_upper_arm_joint" id="12"/>
+      <xacro:feetech_joint joint_name="left_upper_elbow_joint" id="13"/>
+      <xacro:feetech_joint joint_name="left_lower_elbow_joint" id="14"/>
+      <xacro:feetech_joint joint_name="left_forearm_joint" id="15"/>
+      <xacro:feetech_joint joint_name="left_wrist_pitch_joint" id="16"/>
+      <xacro:feetech_joint joint_name="left_wrist_tool_joint" id="17"/>
+      <!-- Right Arm Joints -->
+      <xacro:feetech_joint joint_name="right_shoulder_pitch_joint" id="1"/>
+      <xacro:feetech_joint joint_name="right_upper_arm_joint" id="2"/>
+      <xacro:feetech_joint joint_name="right_upper_elbow_joint" id="3"/>
+      <xacro:feetech_joint joint_name="right_lower_elbow_joint" id="4"/>
+      <xacro:feetech_joint joint_name="right_forearm_joint" id="5"/>
+      <xacro:feetech_joint joint_name="right_wrist_pitch_joint" id="6"/>
+      <xacro:feetech_joint joint_name="right_wrist_tool_joint" id="7"/>
+    </ros2_control>
+  </xacro:macro>
 </robot>

File: wsl_ws/src/moveit_aizee/config/aizee_model.urdf.xacro (robot description, xacro)
@@ -1,4 +1,5 @@
 <?xml version="1.0"?>
 <robot xmlns:xacro="http://www.ros.org/wiki/xacro" name="aizee_model">
+    <xacro:arg name="ros2_control_hardware_type" default="mock_components"/>
     <xacro:arg name="initial_positions_file" default="initial_positions.yaml" />
     <!-- Import aizee_model urdf file -->
@@ -6,4 +7,4 @@
     <!-- Import control_xacro -->
     <xacro:include filename="aizee_model.ros2_control.xacro" />
-    <xacro:aizee_model_ros2_control name="FakeSystem" initial_positions_file="$(arg initial_positions_file)"/>
+    <xacro:aizee_model_ros2_control name="$(arg ros2_control_hardware_type)" initial_positions_file="$(arg initial_positions_file)"/>
 </robot>

Commit message: Actually fixed the joints...

File: wsl_ws/install/moveit_aizee/share/moveit_aizee/config/aizee_model.ros2_control.xacro (robot description, xacro)
@@ -1 +1 @@
-/home/ltr/aizee/wsl_ws/src/moveit_aizee/config/aizee_model.ros2_control.xacro
+/home/skavrx/aizee/wsl_ws/src/moveit_aizee/config/aizee_model.ros2_control.xacro

File: wsl_ws/install/moveit_aizee/share/moveit_aizee/config/aizee_model.urdf.xacro (robot description, xacro)
@@ -1 +1 @@
-/home/ltr/aizee/wsl_ws/src/moveit_aizee/config/aizee_model.urdf.xacro
+/home/skavrx/aizee/wsl_ws/src/moveit_aizee/config/aizee_model.urdf.xacro

File: wsl_ws/src/aizee_model/urdf/aizee_model.urdf (robot description, URDF)
Before this commit: robot aizee_model, 24 links, 23 joints
Joints:
- joint gantry_swivel_joint: type continuous -> revolute
- joint head_pitch_joint: type continuous -> revolute
- joint head_swivel_joint: type continuous -> revolute
- joint head_tilt_joint: type continuous -> revolute
- joint left_forearm_joint: limit lower=-3.14 upper=3.14 effort=1 velocity=1 -> lower=-2.0 upper=2.5 effort=1 velocity=1; type continuous -> revolute
- joint left_lower_elbow_joint: limit lower=-3.14 upper=3.14 effort=1 velocity=1 -> lower=-2.1 upper=0 effort=1 velocity=1; type continuous -> revolute
- joint left_shoulder_pitch_joint: limit lower=-3.14 upper=3.14 effort=1 velocity=1 -> lower=-1.82 upper=1.57 effort=1 velocity=1; type continuous -> revolute
- joint left_upper_arm_joint: axis -0.0539479353612109 0 -0.998543749802813 -> 0.0539479353612109 0 0.998543749802813; limit lower=-3.14 upper=3.14 effort=1 velocity=1 -> lower=-2.7 upper=0 effort=1 velocity=1; type continuous -> revolute
- joint left_upper_elbow_joint: limit lower=-3.14 upper=3.14 effort=1 velocity=1 -> lower=-0.815 upper=1.05 effort=1 velocity=1; type continuous -> revolute
- joint left_wrist_pitch_joint: limit lower=-3.14 upper=3.14 effort=1 velocity=1 -> lower=-0.22 upper=0.22 effort=1 velocity=1; type continuous -> revolute
- joint left_wrist_tool_joint: limit lower=-3.14 upper=3.14 effort=1 velocity=1 -> lower=-1.5 upper=1.5 effort=1 velocity=1; type continuous -> revolute
- joint right_forearm_joint: limit lower=-3.14 upper=3.14 effort=1 velocity=1 -> lower=-2.5 upper=2.0 effort=1 velocity=1; type continuous -> revolute
- joint right_lower_elbow_joint: limit lower=-3.14 upper=3.14 effort=1 velocity=1 -> lower=0 upper=2.1 effort=1 velocity=1; type continuous -> revolute
- joint right_shoulder_pitch_joint: limit lower=-3.14 upper=3.14 effort=1 velocity=1 -> lower=-1.57 upper=1.82 effort=1 velocity=1; type continuous -> revolute
- joint right_upper_arm_joint: axis -0.0539479353612105 0 0.998543749802813 -> 0.0539479353612105 0 -0.998543749802813; limit lower=-3.14 upper=3.14 effort=1 velocity=1 -> lower=0 upper=2.7 effort=1 velocity=1; type continuous -> revolute
- joint right_upper_elbow_joint: limit lower=-3.14 upper=3.14 effort=1 velocity=1 -> lower=-1.05 upper=0.815 effort=1 velocity=1; type continuous -> revolute
- joint right_wrist_pitch_joint: limit lower=-3.14 upper=3.14 effort=1 velocity=1 -> lower=-0.22 upper=0.22 effort=1 velocity=1; type continuous -> revolute
- joint right_wrist_tool_joint: limit lower=-3.14 upper=3.14 effort=1 velocity=1 -> lower=-1.5 upper=1.5 effort=1 velocity=1; type continuous -> revolute
