Commit message: feat(teleop): Meta Quest Pro WebXR teleop + collision-aware IK + URDF refresh
Adds a Cartesian VR teleop path alongside the SO-101 / OpenRB-150 leader
arms.  Drop-in via --leader quest; preserves the existing 30 Hz ZMQ
publish, HDF5 record schema, and gamepad/joystick paths.

New subsystems

  * python/ik/ — URDF parser + FK + Jacobian + 6-DoF DLS IK on aizee.urdf,
    collision-aware joint-limit sweep (trimesh + python-fcl), reachable
    EE workspace AABB computation.  Joint limits write back to YAML and
    overlay into the IK on construction.

  * python/web/ — HTTPS server (aiohttp) + self-signed cert + WebSocket
    pose stream + WebRTC camera bridge (aiortc/PyAV) + in-VR pokable
    button UI.  Includes /preview URDF viewer with slider-bound editable
    joint limits + live mesh collision check, and a standalone
    sim_visual_ik.py for hardware-free development.

  * python/teleop/quest_leader.py — clutched incremental Cartesian leader
    implementing the duck-typed leader interface.  Hand-tracking support
    (index pinch = clutch, middle pinch = gripper), outlier rejection on
    pose jumps, per-joint + Cartesian velocity caps, B-button e-stop with
    dual-grip clear, runtime workspace resize via /api/quest_command.

  * config/quest_teleop.yaml — workspace clamp + IK weights + safety knobs
  * config/joint_limits.yaml — effective joint limits from collision sweep
  * config/joint_align.json — URDF-to-motor frame offsets + signs

URDF refresh (onshape-to-robot re-export)

  * urdf/aizee/aizee.urdf — regenerated from current CAD; wrist_roll
    renamed to wrist_swivel in the URDF.  Codebase/firmware still use
    wrist_roll — they map by position not name, so the rename is
    isolated to the IK + visualization paths.

Plumbing + tuning

  * collect_demo.py / record_replay.py: --leader quest wiring, telem and
    camera-JPEG mirror into the web SharedState
  * requirements.txt: aiohttp, cryptography, aiortc, av
  * firmware/openrb_leader: EMI hardening on the I2C bus
  * rover yaml + leader/robstride calibrations: assorted tuning
  * scripts/aizee-reset-usb-can: USB-CAN reset helper
  * episode_visualizer.py, training/inference.py, viz/: misc tools

Co-Authored-By: Claude Opus 4.7 <noreply@anthropic.com>

File: urdf/aizee/aizee.urdf (robot description, URDF)
Before this commit: robot aizee, 9 links, 8 joints
Links:
- removed link scxxkl_stp
- added link 1_1_02_eb571_960_stp_2, mass 0; collision mesh filename=package://meshes\1_1_02_eb571_960_stp__2.stl; collision mesh filename=package://meshes\1_1_04_eb572_5105_stp__2.stl
- link 1_1_02_eb571_960_stp: geometry collision mesh filename=package://meshes\1_1_02_eb571_960_stp.stl; collision mesh filename=package://meshes\1_1_04_eb572_5105_stp.stl
- link part_33: geometry collision mesh filename=package://meshes\1_1_06_eb673_516_1_stp.stl; collision mesh filename=package://meshes\1_1_06_eb673_524_1_stp.stl
- link part_42: geometry collision mesh filename=package://meshes\1_1_02_eb671_502_1_stp.stl; collision mesh filename=package://meshes\1_1_04_eb672_503_1_stp.stl
Joints:
- removed joint wrist_roll
- added joint wrist_swivel: type revolute, parent 1_1_02_eb571_960_stp, child 1_1_02_eb571_960_stp_2, origin xyz=-0 -0.036 -0.071885 rpy=1.5708 -0 -0, axis 0 0 1, limit lower=-3.141592653589793 upper=3.141592653589793 effort=10 velocity=10
- joint gantry_base: origin xyz=0.0166 0 0.065 rpy=-1.5708 0.00227071 1.5708 -> xyz=0.0166 -0 0.065 rpy=-1.5708 0.00227071 1.5708
- joint gantry_end: origin xyz=-0.562406 -0.0420179 -0.00695 rpy=-0 -0 0.0546306 -> xyz=-0.562406 -0.0420179 -0.00695 rpy=0 0 0.0546306
- joint wrist_pitch: child scxxkl_stp -> 1_1_02_eb571_960_stp; origin xyz=-0.106866 0.00560061 0.0357124 rpy=1.5708 -0 1.51844 -> xyz=-0.11497 0.00602531 0.0357124 rpy=0.0523599 1.5708 0
